File: pcmcia-sram.kicad_pcb (KiCad board)
At the start: 2 copper layers, 110.2 x 87.9 mm, 2 parts, among them J1 Conn_02x34_Top_Bottom, J2 Conn_02x34_Top_Bottom

Commit message: Initial layout
Parts:
- removed J2: Conn_02x34_Top_Bottom, pcmcia:pcmcia_single
- added BT1: Battery, Battery:Battery_Panasonic_CR2032-VS1N_Vertical_CircularHoles, F.Cu at (162.0, 86.2)
- added C1: 0.1uF, Capacitor_SMD:C_0805_2012Metric_Pad1.18x1.45mm_HandSolder, F.Cu at (213.3, 87.0)
- added C2: C_Polarized, Capacitor_SMD:C_1206_3216Metric_Pad1.33x1.80mm_HandSolder, F.Cu at (209.9, 86.8)
- added C3: 0.1uF, Capacitor_SMD:C_0805_2012Metric_Pad1.18x1.45mm_HandSolder, F.Cu at (230.9, 87.0)
- added C4: C_Polarized, Capacitor_SMD:C_1206_3216Metric_Pad1.33x1.80mm_HandSolder, F.Cu at (234.5, 87.0)
- added D1: BAT54C, Package_TO_SOT_SMD:SOT-23, F.Cu at (186.1, 87.8)
- added R1: 10K, Resistor_SMD:R_0805_2012Metric_Pad1.20x1.40mm_HandSolder, F.Cu at (212.7, 92.2)
- added U1: AS6C8008-55ZIN, Package_SO:TSOP-II-44_10.16x18.41mm_P0.8mm, F.Cu at (221.7, 87.0)
- J1: value Conn_02x34_Top_Bottom -> PCMCIA; footprint Connector_PinHeader_2.54mm:PinHeader_2x34_P2.54mm_Vertical -> pcmcia:pcmcia
- moved J1 170.2 mm to (253.9, 87.4)
Connections:
- J1 pad 1: /01 -> GND
- J1 pad 10: /10 -> /A11
- J1 pad 11: /11 -> /A9
- J1 pad 12: /12 -> /A8
- J1 pad 13: /13 -> /A13
- J1 pad 14: /14 -> /A14
- J1 pad 15: /15 -> /WE
- J1 pad 16: /16 -> unconnected-(J1-Pad16)
- J1 pad 17: /17 -> +5V
- J1 pad 18: /18 -> unconnected-(J1-Pad18)
- J1 pad 19: /19 -> /A16
- J1 pad 2: /02 -> /D3
- J1 pad 20: /20 -> /A15
- J1 pad 21: /21 -> /A12
- J1 pad 22: /22 -> /A7
- J1 pad 23: /23 -> /A6
- J1 pad 24: /24 -> /A5
- J1 pad 25: /25 -> /A4
- J1 pad 26: /26 -> /A3
- J1 pad 27: /27 -> /A2
- J1 pad 28: /28 -> /A1
- J1 pad 29: /29 -> /A0
- J1 pad 3: /03 -> /D4
- J1 pad 30: /30 -> /D0
- J1 pad 31: /31 -> /D1
- J1 pad 32: /32 -> /D2
- J1 pad 33: /33 -> +5V
- J1 pad 34: /34 -> GND
- J1 pad 35: /36 -> GND
- J1 pad 36: /37 -> GND
- J1 pad 37: /38 -> unconnected-(J1-Pad37)
- J1 pad 38: /39 -> unconnected-(J1-Pad38)
- J1 pad 39: /40 -> unconnected-(J1-Pad39)
- J1 pad 4: /04 -> /D5
- J1 pad 40: /41 -> unconnected-(J1-Pad40)
- J1 pad 41: /42 -> unconnected-(J1-Pad41)
- J1 pad 42: /43 -> unconnected-(J1-Pad42)
- J1 pad 43: /44 -> unconnected-(J1-Pad43)
- J1 pad 44: /45 -> unconnected-(J1-Pad44)
- J1 pad 45: /46 -> unconnected-(J1-Pad45)
- J1 pad 46: /47 -> /A17
- J1 pad 47: /48 -> /A18
- J1 pad 48: /49 -> /A19
- J1 pad 49: /50 -> unconnected-(J1-Pad49)
- J1 pad 5: /05 -> /D6
- J1 pad 50: /51 -> unconnected-(J1-Pad50)
- J1 pad 51: /52 -> +5V
- J1 pad 52: /53 -> unconnected-(J1-Pad52)
- J1 pad 53: /54 -> unconnected-(J1-Pad53)
- J1 pad 54: /55 -> unconnected-(J1-Pad54)
- J1 pad 55: /56 -> unconnected-(J1-Pad55)
- J1 pad 56: /57 -> unconnected-(J1-Pad56)
- J1 pad 57: /58 -> unconnected-(J1-Pad57)
- J1 pad 58: /59 -> unconnected-(J1-Pad58)
- J1 pad 59: /60 -> unconnected-(J1-Pad59)
- J1 pad 6: /06 -> /D7
- J1 pad 60: /61 -> unconnected-(J1-Pad60)
- J1 pad 61: /62 -> unconnected-(J1-Pad61)
- J1 pad 62: /63 -> unconnected-(J1-Pad62)
- J1 pad 63: /64 -> unconnected-(J1-Pad63)
- J1 pad 64: /65 -> (no net)
- J1 pad 65: /66 -> unconnected-(J1-Pad65)
- J1 pad 66: /67 -> unconnected-(J1-Pad66)
- J1 pad 67: /68 -> GND
- J1 pad 68: /69 -> GND
- J1 pad 7: /07 -> /CE
- J1 pad 8: /08 -> /A10
- J1 pad 9: /09 -> /OE
Routing:
- net /68: track 116.2 -> 0.00 mm
- net /66: track 115.6 -> 0.00 mm
- net /01: track 115.6 -> 0.00 mm
- net /64: track 115.1 -> 0.00 mm
- net /03: track 115.1 -> 0.00 mm
- net /62: track 114.6 -> 0.00 mm
- net /05: track 114.6 -> 0.00 mm
- net /60: track 114.1 -> 0.00 mm
- net /07: track 114.1 -> 0.00 mm
- net /58: track 113.5 -> 0.00 mm
- net /09: track 113.5 -> 0.00 mm
- net /69: track 113.4 -> 0.00 mm
- net /11: track 113.2 -> 0.00 mm
- net /56: track 113.0 -> 0.00 mm
- net /67: track 112.8 -> 0.00 mm
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- added copper zone on In1.Cu, net GND
- added copper zone on In2.Cu, net VCC
Other:
- board outline removed
- copper layers 2 -> 4

Commit message: Various fixes
Parts:
- CR2032: renamed from BT1; footprint Battery:Battery_Panasonic_CR2032-VS1N_Vertical_CircularHoles -> pcmcia:BAT_BAT-HLD-001
- moved CR2032 3.44 mm to (165.5, 86.2)
- moved D1 2.30 mm to (186.3, 85.5)
- moved J1 0.76 mm to (253.9, 88.1)
- moved R1 0.76 mm to (212.0, 92.2)
- turned C1 to -90 degrees
- turned C2 to -90 degrees
Connections:
- J1 pad 64: (no net) -> unconnected-(J1-Pad64)
- U1 pad 39: /A -> /A8
Routing:
- net +5V: track 4.93 -> 99.3 mm
- net /A12: track 0.00 -> 63.7 mm, vias 0 -> 2
- net /A14: track 0.00 -> 61.2 mm, vias 0 -> 2
- net GND: track 19.0 -> 75.2 mm
- net /A13: track 0.00 -> 54.6 mm, vias 0 -> 2
- net /A11: track 0.00 -> 49.4 mm, vias 0 -> 2
- net +BATT: track 0.00 -> 49.3 mm
- net /A9: track 0.00 -> 48.3 mm, vias 0 -> 2
- net /A8: track 0.00 -> 48.3 mm, vias 0 -> 2
- net /OE: track 0.00 -> 47.6 mm, vias 0 -> 2
- net /D2: track 0.00 -> 46.7 mm, vias 0 -> 2
- net /A10: track 0.00 -> 46.2 mm, vias 0 -> 2
- net /D6: track 0.00 -> 44.9 mm
- net /D7: track 0.00 -> 44.6 mm
- net /D4: track 0.00 -> 43.8 mm
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Other:
- board outline added: 94.2 x 50.8 mm

Commit message: Various fixes
Parts:
- moved D1 18.1 mm to (204.3, 87.3), turned to 180 degrees
- moved CR2032 9.61 mm to (174.9, 88.3)
Routing:
- net +BATT: track 49.3 -> 68.9 mm
- net VCC: track 19.7 -> 33.1 mm, vias 5 -> 2
- net +5V: track 99.3 -> 89.8 mm, vias 0 -> 2
- added copper zone on B.Cu, net GND
- removed copper zone on In1.Cu, net GND
- removed copper zone on In2.Cu, net VCC
Other:
- board size 94.2 x 50.8 mm -> 84.7 x 50.8 mm
- copper layers 4 -> 2
- board text added: "1024KB"
- board text added: "8-bit SRAM"
- board text added: "CR2032"
- board text added: "Version 1.0 (Dec 2023)"
- board text added: "https://retro.engineer"
