File: pcmcia-sram.kicad_pcb (KiCad board)
At the start: 2 copper layers, 84.7 x 50.8 mm, 8 parts, among them J1 PCMCIA, U1 AS6C8008-55ZIN

Commit message: Revision 1.1
Parts:
- removed R1: 10K, Resistor_SMD:R_0805_2012Metric_Pad1.20x1.40mm_HandSolder
- moved U1 10.6 mm to (211.2, 88.0)
- moved C3 10.6 mm to (219.2, 88.2)
- moved C1 10.0 mm to (203.3, 88.1)
- moved C2 9.03 mm to (200.9, 88.1)
- moved D1 6.92 mm to (197.4, 88.2)
Routing:
- net GND: track 68.6 -> 16.8 mm, vias 8 -> 57
- net /CE: track 38.2 -> 66.9 mm
- net /D3: track 43.1 -> 68.5 mm
- net /A15: track 33.1 -> 53.2 mm
- net +BATT: track 68.9 -> 48.8 mm, vias 0 -> 3
- net /A16: track 32.0 -> 50.6 mm
- net /A19: track 26.0 -> 41.1 mm
- net /WE: track 25.2 -> 39.9 mm, vias 0 -> 2
- net /D7: track 45.5 -> 59.3 mm, vias 0 -> 2
- net /A17: track 26.1 -> 39.2 mm
- net /D6: track 45.9 -> 59.0 mm, vias 0 -> 2
- net /OE: track 48.6 -> 61.0 mm
- net /A18: track 25.8 -> 38.1 mm
- net /D5: track 44.5 -> 56.7 mm, vias 0 -> 2
- net /D4: track 44.8 -> 56.4 mm, vias 0 -> 2
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- added copper zone on F.Cu, net GND
Other:
- board text added: "1024K x 8 bits"
- board text added: "Revision 1.1 (Dec 2023)"
- board text removed: "1024KB"
- board text removed: "8-bit SRAM"
- board text removed: "CR2032"
- board text removed: "Version 1.0 (Dec 2023)"
