File: pcmcia-sram copy.kicad_pcb (KiCad board)
At the start: 2 copper layers, 84.7 x 50.8 mm, 8 parts, among them J1 PCMCIA, U1 AS6C8008-55ZIN

Commit message: Add new design
Parts:
- moved C2 22.1 mm to (231.9, 87.0), turned to 90 degrees
- moved D1 4.57 mm to (208.9, 87.2)
Routing:
- net GND: track 68.6 -> 15.8 mm, vias 8 -> 31
- net /CE: track 38.2 -> 55.9 mm
- net /A13: track 53.4 -> 37.6 mm
- net /D3: track 43.1 -> 57.5 mm
- net /A14: track 53.4 -> 39.9 mm
- net /A12: track 62.1 -> 48.6 mm, vias 2 -> 4
- net /A15: track 33.1 -> 43.7 mm
- net /A9: track 47.4 -> 37.7 mm
- net /A11: track 46.5 -> 37.3 mm
- net /A16: track 32.0 -> 39.9 mm
- net +BATT: track 68.9 -> 63.6 mm, vias 0 -> 3
- net /A8: track 50.3 -> 45.0 mm
- net /A10: track 43.9 -> 39.3 mm
- net /A19: track 26.0 -> 30.5 mm
- net /WE: track 25.2 -> 29.4 mm, vias 0 -> 2
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- added copper zone on F.Cu, net GND
Other:
- board text added: "1024K x 8 bits"
- board text added: "Version 1.1 (Dec 2023)"
- board text removed: "1024KB"
- board text removed: "8-bit SRAM"
- board text removed: "CR2032"
- board text removed: "Version 1.0 (Dec 2023)"
